File: hw/drone.kicad_pcb (KiCad board)
At the start: 2 copper layers, 26 parts, among them J1 CONN_20, J2 CONN_20, M1 ANTENNAGPS-2X7MM, U1 CC1101RGPR, U2 LSM9DS1TR, Y1 CRYSTALPTH-2X6

Commit message: Partial start to PCB layout.
Parts:
- moved Y1 12.5 mm to (129.8, 100.6)
- moved M1 12.5 mm to (136.1, 81.8)
- moved C14 8.21 mm to (186.2, 72.4), turned to 180 degrees
- moved C12 7.43 mm to (188.7, 69.3), turned to 180 degrees
- moved C10 2.78 mm to (185.7, 64.0), turned to 180 degrees
- moved C13 2.45 mm to (189.5, 70.9), turned to 180 degrees
- moved C11 2.44 mm to (185.4, 69.6), turned to 180 degrees
- moved U2 1.61 mm to (178.1, 65.5)
Connections:
- U2 pad 2: /IMU/IMU_SCK -> /A5
- U2 pad 4: /B13 -> /A7
- U2 pad 5: /IMU/IMU_MISO -> /A6
- U2 pad 6: /IMU/IMU_MISO -> /A6
- U2 pad 7: /IMU/IMU_CS -> /A3
- U2 pad 8: /IMU/MAG_CS -> /A2
Routing:
- net GND: track 0.00 -> 5.00 mm
- net /A6: track 0.00 -> 0.59 mm
- added copper zone on F.Cu, net 3.3V
- added copper zone on B.Cu, net GND
Other:
- board outline added: 62.2 x 25.4 mm
